Commit message: small changes to headers

File: kart_description/urdf/kart.xacro (robot description, xacro)
@@ -1,7 +1,4 @@
 <?xml version="1.0"?>
 <robot name="kart" xmlns:xacro="http://www.ros.org/wiki/xacro">
-	<xacro:include filename="$(find kart_description)/urdf/kart.gazebo" />
-	<xacro:include filename="$(find kart_description)/urdf/materials.xacro" />
-	<xacro:include filename="$(find kart_description)/urdf/macros.xacro" />
         <!-- Put here the robot description -->
 	<xacro:property name="PI" value="3.1415926535897931"/>
@@ -18,4 +15,7 @@
 	<xacro:property name="cameraSize" value="0.05"/>
 	<xacro:property name="cameraMass" value="0.1"/>
+	<xacro:include filename="$(find kart_description)/urdf/kart.gazebo" />
+	<xacro:include filename="$(find kart_description)/urdf/materials.xacro" />
+	<xacro:include filename="$(find kart_description)/urdf/macros.xacro" />
 	<link name="footprint" />
 	<joint name="base_joint" type="fixed">
@@ -67,3 +67,5 @@
 	  </inertial>
 	</link>
+	<wheel lr="left" tY="1"/>
+	<wheel lr="right" tY="-1"/>
 </robot>

File: kart_description/urdf/macros.xacro (robot description, xacro)
@@ -1,4 +1,4 @@
 <?xml version="1.0"?>
-<robot name="kart" xmlns:xacro="http://www.ros.org/wiki/xacro">
+<robot>
         <!-- Put here the robot description -->
 	<macro name="cylinder_inertia" params="m r h">
@@ -59,5 +59,7 @@
 	<transmission name="${lr}_trans">
 	  <type>transmission_interface/SimpleTransmission</type>
-	  <joint name="${lr}_wheel_hinge"/>
+	  <joint name="${lr}_wheel_hinge">
+		<hardwareInterface>EffortJointInterface</hardwareInterface>
+	  </joint>
 	  <actuator name="${lr}Motor">
 	    <hardwareInterface>EffortJointInterface</hardwareInterface>

File: kart_description/urdf/materials.xacro (robot description, xacro)
@@ -1,4 +1,4 @@
 <?xml version="1.0"?>
-<robot name="kart" xmlns:xacro="http://www.ros.org/wiki/xacro">
+<robot>
         <!-- Put here the robot description -->
 	<material name="black">
